File: meltybrain/Eagle_CAD/Hocki_IR_Receiver/Hocki-IR-Receiver.sch (EAGLE design)
At the start: 71 parts, among them J1 SM03B-SRSS-TB(LF)(SN), U1 OPA2380AIDGKR, U10 NL27WZ32USG, U11 TMUX1204DGSR, U2 OPA2380AIDGKR, U3 AP2210K-5.0TRG1, U4 LMH6612MAX/NOPB, U5 LMH6612MAX/NOPB, U7 TLV3502AIDCNR, U8 TLV3502AIDCNR, U9 SN74LVC1G58DCKR

Commit message: added current draws to ir board
Other:
- note added: "5V total current: 151.52mA regulator rating: 300mA also has overcurrent, overtemperature, and reverse polarity protections"
- note added: "Current: 0.13mA worst case total: 0.4mA"
- note added: "Current: 0.5mA configurable logic 0.01mA per OR gate total: 0.52mA"
- note added: "Current: 10mA per pulldown mux very low total: 40mA"
- note added: "Current: 15mA for 9V LED 11mA for 5V LED"
- note added: "Current: 1mA voltage divider 10mA per op-amp total: 42mA"
- note added: "Current: 3.9mA per opamp 10mA for voltage divider total: 25.6mA"
- note added: "Current: 5mA per comparator 2mA for voltage divider 10mA termination total: 32mA"
- moved on the sheet: C1, C10, C13, C14, C15, C16, C17, C2, C3, C4, C5, C6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
