File: meltybrain/Eagle_CAD/LED_Board/LED_BOARD.brd (EAGLE design)
At the start: 56 x 12 mm, 17 parts, among them J1 SM04B-SRSS-TB(LF)(SN), U1 DOTSTAR, U2 DOTSTAR, U3 DOTSTAR, U4 DOTSTAR, U5 DOTSTAR, U6 DOTSTAR, U7 DOTSTAR, U8 DOTSTAR

Commit message: Changes to LED board
Parts:
- moved C8 2.06 mm to (4.00, 2.00)
- moved C1 2.00 mm to (52.5, 2.00)
- moved C2 2.00 mm to (47.5, 2.00)
- moved C3 2.00 mm to (36.5, 2.00)
- moved C4 2.00 mm to (31.5, 2.00)
- moved C5 2.00 mm to (24.5, 2.00)
- moved C6 2.00 mm to (19.5, 2.00)
- moved C7 2.00 mm to (8.50, 2.00)
- moved J1 2.00 mm to (5.00, 6.00)
- moved U1 2.00 mm to (52.5, 9.00)
- moved U2 2.00 mm to (45.5, 9.00)
- moved U3 2.00 mm to (38.5, 9.00)
- moved U4 2.00 mm to (31.5, 9.00)
- moved U5 2.00 mm to (24.5, 9.00)
- moved U6 2.00 mm to (17.5, 9.00)
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Connections:
- net +5V: no longer J1.S1, J1.S2
- net GND: now also J1.S1, J1.S2
Routing:
- net +5V: track 12.0 -> 2.00 mm
